File: RIAA_preamp.kicad_pcb (KiCad board)
At the start: 2 copper layers, 94 x 50 mm, 130 parts, among them J1 Conn_01x02, J2 Conn_01x02, J3 Conn_01x03, J4 Conn_01x02, T1 BV302D18028, U1 NE5532, U3 MC78M15_TO252, U4 MC79M15_TO252, U5 NE5532

Commit message: WIP
Other:
- board text added: "+"
- board text added: "-"
- board text added: "~"
Changed lines of the file:
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@@
+		)
+	)
+	(gr_text "-"
+		(at 109.3234 48.045 0)
+		(layer "F.SilkS")
+		(effects
+			(font
+				(size 1 1)
+				(thickness 0.1)
+			)
+			(justify left bottom)
 		)
 	)
@@
 			(font
 				(size 0.8 0.8)
+				(thickness 0.1)
+			)
+			(justify left bottom)
+		)
+	)
+	(gr_text "+"
+		(at 109.2726 50.839 0)
+		(layer "F.SilkS")
+		(effects
+			(font
+				(size 1 1)
+				(thickness 0.1)
+			)
+			(justify left bottom)
+		)
+	)
+	(gr_text "~"
+		(at 103.3036 50.7374 0)
+		(layer "F.SilkS")
+		(effects
+			(font
+				(size 1 1)
 				(thickness 0.1)
 			)
@@
 			)
 			(justify left bottom)
+		)
+	)
+	(gr_text "~"
+		(at 103.329 48.045 0)
+		(layer "F.SilkS")
+		(effects
+			(font
+				(size 1 1)
+				(thickness 0.1)
+			)
+			(justify left bottom)
